Commit message: Added passing joints as argument

File: model/model.urdf (robot description, URDF)
Before this commit: robot iCub, 189 links, 188 joints
Links:
- removed link l_sole_skin_0
- removed link l_sole_skin_1
- removed link l_sole_skin_10
- removed link l_sole_skin_11
- removed link l_sole_skin_12
- removed link l_sole_skin_13
- removed link l_sole_skin_14
- removed link l_sole_skin_15
- removed link l_sole_skin_17
- removed link l_sole_skin_18
- removed link l_sole_skin_19
- removed link l_sole_skin_2
- removed link l_sole_skin_20
- removed link l_sole_skin_21
- removed link l_sole_skin_22
- removed link l_sole_skin_24
- removed link l_sole_skin_25
- removed link l_sole_skin_26
- removed link l_sole_skin_27
- removed link l_sole_skin_28
- removed link l_sole_skin_29
- removed link l_sole_skin_3
- removed link l_sole_skin_4
- removed link l_sole_skin_8
- removed link l_sole_skin_9
- removed link r_sole_skin_0
- removed link r_sole_skin_1
- removed link r_sole_skin_10
- removed link r_sole_skin_11
- removed link r_sole_skin_12
- removed link r_sole_skin_13
- removed link r_sole_skin_14
- removed link r_sole_skin_15
- removed link r_sole_skin_17
- removed link r_sole_skin_18
- removed link r_sole_skin_19
- removed link r_sole_skin_2
- removed link r_sole_skin_20
- removed link r_sole_skin_21
- removed link r_sole_skin_22
- removed link r_sole_skin_24
- removed link r_sole_skin_25
- removed link r_sole_skin_26
- removed link r_sole_skin_27
- removed link r_sole_skin_28
- removed link r_sole_skin_29
- removed link r_sole_skin_3
- removed link r_sole_skin_4
- removed link r_sole_skin_8
- removed link r_sole_skin_9
- added link root_link_imu_frame
- link chest: geometry collision mesh filename=package://iCub/meshes/simmechanics/2-5_plus/sim_sea_2-5_che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 scale=0.001 0.001 0.001; visual mesh filename=package://iCub/meshes/simmechanics/2-5_plus/sim_sea_2-5_che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 scale=0.001 0.001 0.001
- link head: geometry collision mesh filename=package://iCub/meshes/simmechanics/2-5_plus/sim_sea_2-5_hea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 scale=0.001 0.001 0.001; visual mesh filename=package://iCub/meshes/simmechanics/2-5_plus/sim_sea_2-5_hea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 scale=0.001 0.001 0.001
- link l_ankle_1: geometry collision mesh filename=package://iCub/meshes/simmechanics/2-5_plus/sim_sea_2-5_l_a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 scale=0.001 0.001 0.001; visual mesh filename=package://iCub/meshes/simmechanics/2-5_plus/sim_sea_2-5_l_a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 scale=0.001 0.001 0.001
- link l_ankle_2: mass 0.265122 -> 0.265337; geometry collision mesh filename=package://iCub/meshes/simmechanics/2-5_plus/sim_sea_2-5_l_f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 scale=0.001 0.001 0.001; visual mesh filename=package://iCub/meshes/simmechanics/2-5_plus/sim_sea_2-5_l_f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 scale=0.001 0.001 0.001
- link l_elbow_1: geometry collision mesh filename=package://iCub/meshes/simmechanics/2-5_plus/sim_sea_2-5_l_e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 scale=0.001 0.001 0.001; visual mesh filename=package://iCub/meshes/simmechanics/2-5_plus/sim_sea_2-5_l_e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 scale=0.001 0.001 0.001
- link l_foot: mass 0.382968 -> 0.357881; geometry collision mesh filename=package://iCub/meshes/simmechanics/2-5_plus/sim_sea_2-5_l_s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 scale=0.001 0.001 0.001; visual mesh filename=package://iCub/meshes/simmechanics/2-5_plus/sim_sea_2-5_l_s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 scale=0.001 0.001 0.001
- link l_forearm: geometry collision mesh filename=package://iCub/meshes/simmechanics/2-5_plus/sim_sea_2-5_l_f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 scale=0.001 0.001 0.001; visual mesh filename=package://iCub/meshes/simmechanics/2-5_plus/sim_sea_2-5_l_f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 scale=0.001 0.001 0.001
- link l_hand: geometry collision mesh filename=package://iCub/meshes/simmechanics/2-5_plus/sim_sea_2-5_l_h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 scale=0.001 0.001 0.001; visual mesh filename=package://iCub/meshes/simmechanics/2-5_plus/sim_sea_2-5_l_h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 scale=0.001 0.001 0.001
- link l_hip_1: geometry collision mesh filename=package://iCub/meshes/simmechanics/2-5_plus/sim_sea_2-5_l_h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 scale=0.001 0.001 0.001; visual mesh filename=package://iCub/meshes/simmechanics/2-5_plus/sim_sea_2-5_l_h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 scale=0.001 0.001 0.001
- link l_hip_2: mass 0.415987 -> 0.421106; geometry collision mesh filename=package://iCub/meshes/simmechanics/2-5_plus/sim_sea_2-5_l_h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 scale=0.001 0.001 0.001; visual mesh filename=package://iCub/meshes/simmechanics/2-5_plus/sim_sea_2-5_l_h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 scale=0.001 0.001 0.001
- link l_hip_3: geometry collision mesh filename=package://iCub/meshes/simmechanics/2-5_plus/sim_sea_2-5_l_u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 scale=0.001 0.001 0.001; visual mesh filename=package://iCub/meshes/simmechanics/2-5_plus/sim_sea_2-5_l_u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 scale=0.001 0.001 0.001
- link l_lower_leg: geometry collision mesh filename=package://iCub/meshes/simmechanics/2-5_plus/sim_sea_2-5_l_s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 scale=0.001 0.001 0.001; visual mesh filename=package://iCub/meshes/simmechanics/2-5_plus/sim_sea_2-5_l_s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 scale=0.001 0.001 0.001
- link l_shoulder_1: geometry collision mesh filename=package://iCub/meshes/simmechanics/2-5_plus/sim_sea_2-5_l_s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 scale=0.001 0.001 0.001; visual mesh filename=package://iCub/meshes/simmechanics/2-5_plus/sim_sea_2-5_l_s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 scale=0.001 0.001 0.001
- link l_shoulder_2: geometry collision mesh filename=package://iCub/meshes/simmechanics/2-5_plus/sim_sea_2-5_l_s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 scale=0.001 0.001 0.001; visual mesh filename=package://iCub/meshes/simmechanics/2-5_plus/sim_sea_2-5_l_s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 scale=0.001 0.001 0.001
- link l_shoulder_3: geometry collision mesh filename=package://iCub/meshes/simmechanics/2-5_plus/sim_sea_2-5_l_u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 scale=0.001 0.001 0.001; visual mesh filename=package://iCub/meshes/simmechanics/2-5_plus/sim_sea_2-5_l_u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 scale=0.001 0.001 0.001
- link l_upper_arm: geometry collision mesh filename=package://iCub/meshes/simmechanics/2-5_plus/sim_sea_2-5_l_e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 scale=0.001 0.001 0.001; visual mesh filename=package://iCub/meshes/simmechanics/2-5_plus/sim_sea_2-5_l_e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 scale=0.001 0.001 0.001
- link l_upper_leg: geometry collision mesh filename=package://iCub/meshes/simmechanics/2-5_plus/sim_sea_2-5_l_t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 scale=0.001 0.001 0.001; visual mesh filename=package://iCub/meshes/simmechanics/2-5_plus/sim_sea_2-5_l_t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 scale=0.001 0.001 0.001
- link l_wrist_1: geometry collision mesh filename=package://iCub/meshes/simmechanics/2-5_plus/sim_sea_2-5_l_w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 scale=0.001 0.001 0.001; visual mesh filename=package://iCub/meshes/simmechanics/2-5_plus/sim_sea_2-5_l_w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 scale=0.001 0.001 0.001
- link neck_1: geometry collision mesh filename=package://iCub/meshes/simmechanics/2-5_plus/sim_sea_2-5_nec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 scale=0.001 0.001 0.001; visual mesh filename=package://iCub/meshes/simmechanics/2-5_plus/sim_sea_2-5_nec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 scale=0.001 0.001 0.001
- link neck_2: geometry collision mesh filename=package://iCub/meshes/simmechanics/2-5_plus/sim_sea_2-5_nec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 scale=0.001 0.001 0.001; visual mesh filename=package://iCub/meshes/simmechanics/2-5_plus/sim_sea_2-5_nec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 scale=0.001 0.001 0.001
- link r_ankle_1: geometry collision mesh filename=package://iCub/meshes/simmechanics/2-5_plus/sim_sea_2-5_r_a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 scale=0.001 0.001 0.001; visual mesh filename=package://iCub/meshes/simmechanics/2-5_plus/sim_sea_2-5_r_a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 scale=0.001 0.001 0.001
- link r_ankle_2: mass 0.265122 -> 0.265337; geometry collision mesh filename=package://iCub/meshes/simmechanics/2-5_plus/sim_sea_2-5_r_f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 scale=0.001 0.001 0.001; visual mesh filename=package://iCub/meshes/simmechanics/2-5_plus/sim_sea_2-5_r_f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 scale=0.001 0.001 0.001
- link r_elbow_1: geometry collision mesh filename=package://iCub/meshes/simmechanics/2-5_plus/sim_sea_2-5_r_e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 scale=0.001 0.001 0.001; visual mesh filename=package://iCub/meshes/simmechanics/2-5_plus/sim_sea_2-5_r_e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 scale=0.001 0.001 0.001
- link r_foot: mass 0.382866 -> 0.357881; geometry collision mesh filename=package://iCub/meshes/simmechanics/2-5_plus/sim_sea_2-5_r_s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 scale=0.001 0.001 0.001; visual mesh filename=package://iCub/meshes/simmechanics/2-5_plus/sim_sea_2-5_r_s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 scale=0.001 0.001 0.001
- link r_forearm: geometry collision mesh filename=package://iCub/meshes/simmechanics/2-5_plus/sim_sea_2-5_r_f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 scale=0.001 0.001 0.001; visual mesh filename=package://iCub/meshes/simmechanics/2-5_plus/sim_sea_2-5_r_f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 scale=0.001 0.001 0.001
- link r_hand: geometry collision mesh filename=package://iCub/meshes/simmechanics/2-5_plus/sim_sea_2-5_r_h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 scale=0.001 0.001 0.001; visual mesh filename=package://iCub/meshes/simmechanics/2-5_plus/sim_sea_2-5_r_h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 scale=0.001 0.001 0.001
- link r_hip_1: geometry collision mesh filename=package://iCub/meshes/simmechanics/2-5_plus/sim_sea_2-5_r_h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 scale=0.001 0.001 0.001; visual mesh filename=package://iCub/meshes/simmechanics/2-5_plus/sim_sea_2-5_r_h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 scale=0.001 0.001 0.001
- link r_hip_2: mass 0.413242 -> 0.418361; geometry collision mesh filename=package://iCub/meshes/simmechanics/2-5_plus/sim_sea_2-5_r_h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 scale=0.001 0.001 0.001; visual mesh filename=package://iCub/meshes/simmechanics/2-5_plus/sim_sea_2-5_r_h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 scale=0.001 0.001 0.001
- link r_hip_3: geometry collision mesh filename=package://iCub/meshes/simmechanics/2-5_plus/sim_sea_2-5_r_u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 scale=0.001 0.001 0.001; visual mesh filename=package://iCub/meshes/simmechanics/2-5_plus/sim_sea_2-5_r_u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 scale=0.001 0.001 0.001
- link r_lower_leg: geometry collision mesh filename=package://iCub/meshes/simmechanics/2-5_plus/sim_sea_2-5_r_s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 scale=0.001 0.001 0.001; visual mesh filename=package://iCub/meshes/simmechanics/2-5_plus/sim_sea_2-5_r_s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 scale=0.001 0.001 0.001
- link r_shoulder_1: geometry collision mesh filename=package://iCub/meshes/simmechanics/2-5_plus/sim_sea_2-5_r_s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 scale=0.001 0.001 0.001; visual mesh filename=package://iCub/meshes/simmechanics/2-5_plus/sim_sea_2-5_r_s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 scale=0.001 0.001 0.001
- link r_shoulder_2: geometry collision mesh filename=package://iCub/meshes/simmechanics/2-5_plus/sim_sea_2-5_r_s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 scale=0.001 0.001 0.001; visual mesh filename=package://iCub/meshes/simmechanics/2-5_plus/sim_sea_2-5_r_s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 scale=0.001 0.001 0.001
- link r_shoulder_3: geometry collision mesh filename=package://iCub/meshes/simmechanics/2-5_plus/sim_sea_2-5_r_u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 scale=0.001 0.001 0.001; visual mesh filename=package://iCub/meshes/simmechanics/2-5_plus/sim_sea_2-5_r_u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 scale=0.001 0.001 0.001
- link r_upper_arm: geometry collision mesh filename=package://iCub/meshes/simmechanics/2-5_plus/sim_sea_2-5_r_e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 scale=0.001 0.001 0.001; visual mesh filename=package://iCub/meshes/simmechanics/2-5_plus/sim_sea_2-5_r_e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 scale=0.001 0.001 0.001
- link r_upper_leg: geometry collision mesh filename=package://iCub/meshes/simmechanics/2-5_plus/sim_sea_2-5_r_t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 scale=0.001 0.001 0.001; visual mesh filename=package://iCub/meshes/simmechanics/2-5_plus/sim_sea_2-5_r_t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 scale=0.001 0.001 0.001
- link r_wrist_1: geometry collision mesh filename=package://iCub/meshes/simmechanics/2-5_plus/sim_sea_2-5_r_w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 scale=0.001 0.001 0.001; visual mesh filename=package://iCub/meshes/simmechanics/2-5_plus/sim_sea_2-5_r_w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 scale=0.001 0.001 0.001
- link root_link: mass 5.09143 -> 5.12739; geometry collision mesh filename=package://iCub/meshes/simmechanics/2-5_plus/sim_sea_2-5_roo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 scale=0.001 0.001 0.001; visual mesh filename=package://iCub/meshes/simmechanics/2-5_plus/sim_sea_2-5_roo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 scale=0.001 0.001 0.001
- link torso_1: geometry collision mesh filename=package://iCub/meshes/simmechanics/2-5_plus/sim_sea_2-5_lap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 scale=0.001 0.001 0.001; visual mesh filename=package://iCub/meshes/simmechanics/2-5_plus/sim_sea_2-5_lap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 scale=0.001 0.001 0.001
- link torso_2: geometry collision mesh filename=package://iCub/meshes/simmechanics/2-5_plus/sim_sea_2-5_lap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 scale=0.001 0.001 0.001; visual mesh filename=package://iCub/meshes/simmechanics/2-5_plus/sim_sea_2-5_lap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 scale=0.001 0.001 0.001
Joints:
- removed joint l_sole_skin_0_fixed_joint
- removed joint l_sole_skin_10_fixed_joint
- removed joint l_sole_skin_11_fixed_joint
- removed joint l_sole_skin_12_fixed_joint
- removed joint l_sole_skin_13_fixed_joint
- removed joint l_sole_skin_14_fixed_joint
- removed joint l_sole_skin_15_fixed_joint
- removed joint l_sole_skin_17_fixed_joint
- removed joint l_sole_skin_18_fixed_joint
- removed joint l_sole_skin_19_fixed_joint
- removed joint l_sole_skin_1_fixed_joint
- removed joint l_sole_skin_20_fixed_joint
- removed joint l_sole_skin_21_fixed_joint
- removed joint l_sole_skin_22_fixed_joint
- removed joint l_sole_skin_24_fixed_joint
- removed joint l_sole_skin_25_fixed_joint
- removed joint l_sole_skin_26_fixed_joint
- removed joint l_sole_skin_27_fixed_joint
- removed joint l_sole_skin_28_fixed_joint
- removed joint l_sole_skin_29_fixed_joint
- removed joint l_sole_skin_2_fixed_joint
- removed joint l_sole_skin_3_fixed_joint
- removed joint l_sole_skin_4_fixed_joint
- removed joint l_sole_skin_8_fixed_joint
- removed joint l_sole_skin_9_fixed_joint
- removed joint r_sole_skin_0_fixed_joint
- removed joint r_sole_skin_10_fixed_joint
- removed joint r_sole_skin_11_fixed_joint
- removed joint r_sole_skin_12_fixed_joint
- removed joint r_sole_skin_13_fixed_joint
- removed joint r_sole_skin_14_fixed_joint
- removed joint r_sole_skin_15_fixed_joint
- removed joint r_sole_skin_17_fixed_joint
- removed joint r_sole_skin_18_fixed_joint
- removed joint r_sole_skin_19_fixed_joint
- removed joint r_sole_skin_1_fixed_joint
- removed joint r_sole_skin_20_fixed_joint
- removed joint r_sole_skin_21_fixed_joint
- removed joint r_sole_skin_22_fixed_joint
- removed joint r_sole_skin_24_fixed_joint
- removed joint r_sole_skin_25_fixed_joint
- removed joint r_sole_skin_26_fixed_joint
- removed joint r_sole_skin_27_fixed_joint
- removed joint r_sole_skin_28_fixed_joint
- removed joint r_sole_skin_29_fixed_joint
- removed joint r_sole_skin_2_fixed_joint
- removed joint r_sole_skin_3_fixed_joint
- removed joint r_sole_skin_4_fixed_joint
- removed joint r_sole_skin_8_fixed_joint
- removed joint r_sole_skin_9_fixed_joint
- added joint root_link_imu_frame_fixed_joint: type fixed, parent root_link, child root_link_imu_frame, origin xyz=0.08515499999999998 -0.011000000000000022 -0.11230899999999999 rpy=-2.0943952105869323 0 -1.5707963267948963
- joint l_ankle_pitch: axis 2.220446049250313e-16 0.9999999999999998 0.0 -> -6.661338147750939e-16 1.0000000000000002 4.440892098500626e-16; limit lower=-0.6108652381980153 upper=0.6108652381980153 effort=37.0 velocity=7.64 -> lower=-0.8726646259971648 upper=0.3490658503988659 effort=37.0 velocity=7.64; origin xyz=0 0 -0.20049999999999996 rpy=0 0 0 -> xyz=0 0 -0.20049999999999996 rpy=0 0.2617991794798451 0
- joint l_ankle_roll: axis 0.9999999999999998 0.0 2.220446049250313e-16 -> 1.0000001561184808 6.013654019199066e-16 -1.197939497389039e-07
- joint l_foot_ft_sensor: origin xyz=-0.003500000000000003 0 -0.0605 rpy=3.141592653589793 0 0 -> xyz=-0.0034999280659716164 0 -0.060500343280208146 rpy=-3.141592643239301 0 0
- joint l_leg_ft_sensor: origin xyz=-0.0008301999999999962 7.519999999999749e-05 -0.07429999999999995 rpy=3.141592653589793 0 0 -> xyz=-0.0008575000000000041 0 -0.07429999999999995 rpy=3.141592653589793 0 0
- joint l_sole_fixed_joint: origin xyz=0.003500000000000003 0 0.0040000000000000036 rpy=-3.141592653589793 0 0 -> xyz=0.021450226059648844 0 0.006691276652475486 rpy=-3.1415926535897634 0.2617991920983335 0
- joint l_upper_leg_back_contact_fixed_joint: origin xyz=-0.051256699999999995 0 0.014599999999999946 rpy=0 1.5707963267948963 0 -> xyz=-0.05125669999999998 0 0.014599999999999946 rpy=0 1.5707963267948963 0
- joint r_ankle_pitch: axis 2.220446049250313e-16 0.9999999999999998 0.0 -> -6.661338147750939e-16 1.0000000000000002 4.440892098500626e-16; limit lower=-0.6108652381980153 upper=0.6108652381980153 effort=37.0 velocity=7.64 -> lower=-0.8726646259971648 upper=0.3490658503988659 effort=37.0 velocity=7.64; origin xyz=0 0 -0.20049999999999996 rpy=0 0 0 -> xyz=0 0 -0.20049999999999996 rpy=0 0.2617991794798451 0
- joint r_ankle_roll: axis -0.9999999999999998 0.0 -2.220446049250313e-16 -> -1.0000001561184808 -6.013654019199066e-16 1.197939497389039e-07
- joint r_foot_ft_sensor: origin xyz=-0.003500000000000003 0 -0.0605 rpy=3.141592653589793 0 0 -> xyz=-0.0034999280659716164 0 -0.060500343280208146 rpy=3.141592652417863 0 0
- joint r_leg_ft_sensor: origin xyz=-0.0009362999999999941 1.3899999999969492e-05 -0.07429999999999995 rpy=3.141592653589793 0 0 -> xyz=-0.0008575000000000041 0 -0.07429999999999995 rpy=3.141592653589793 0 0
- joint r_lower_leg_skin_0_fixed_joint: origin xyz=0.05441169999999998 -0.03121489999999999 -0.002634000000000025 rpy=2.0917380908554746e-06 -1.4153067624694633 2.48648458622082 -> xyz=0.054411699999999986 -0.031213999999999992 -0.002634000000000025 rpy=2.0917380908554746e-06 -1.4153067624694633 2.48648458622082
- joint r_lower_leg_skin_10_fixed_joint: origin xyz=0.06446069999999998 0.00034239999999997883 -0.021204999999999974 rpy=3.141592653553929 -1.4709580354104241 0.00043002167526072775 -> xyz=0.0644607 0.00034239999999997883 -0.021204999999999974 rpy=3.141592653553929 -1.4709580354104241 0.00043002167526072775
- joint r_lower_leg_skin_11_fixed_joint: origin xyz=0.060710799999999975 -0.016091600000000025 -0.030884999999999996 rpy=-3.1415921825227295 -1.32811804060386 -0.27213836787954737 -> xyz=0.06071079999999999 -0.01609160000000001 -0.030884999999999996 rpy=-3.1415921825227295 -1.32811804060386 -0.27213836787954737
- joint r_lower_leg_skin_14_fixed_joint: origin xyz=0.05504769999999998 -0.031175900000000006 -0.02190000000000003 rpy=-3.1415918188482506 -1.46502735635212 -0.6540334071673009 -> xyz=0.05504769999999999 -0.03117600000000001 -0.02190000000000003 rpy=-3.1415918188482506 -1.46502735635212 -0.6540334071673009
- joint r_lower_leg_skin_15_fixed_joint: origin xyz=0.05917079999999998 -0.016178800000000007 0.0072429999999999994 rpy=4.274842569949443e-07 -1.2520363307607896 2.8679885947088186 -> xyz=0.05917079999999999 -0.016178800000000007 0.0072429999999999994 rpy=4.274842569949443e-07 -1.2520363307607896 2.8679885947088186
- joint r_lower_leg_skin_16_fixed_joint: origin xyz=0.027287599999999978 -0.050286899999999995 -0.004549000000000025 rpy=1.3307591512293707e-05 -1.5326085351498482 1.9628024283508803 -> xyz=0.027287499999999985 -0.050287 -0.004549000000000025 rpy=1.3307591512293707e-05 -1.5326085351498482 1.9628024283508803
- joint r_lower_leg_skin_17_fixed_joint: origin xyz=0.027874999999999976 -0.05031190000000001 -0.023882000000000014 rpy=-3.141564526201752 -1.563662402374811 -1.1802250875588731 -> xyz=0.027874999999999987 -0.05031200000000001 -0.023882000000000014 rpy=-3.141564526201752 -1.563662402374811 -1.1802250875588731
- joint r_lower_leg_skin_19_fixed_joint: origin xyz=0.03575341 0.041062799999999997 0.006064999999999987 rpy=-8.908777145556939e-07 -1.434986969778283 -2.158636180167247 -> xyz=0.035753400000000005 0.04106279999999999 0.006064999999999987 rpy=-8.908777145556939e-07 -1.434986969778283 -2.158636180167247
- joint r_lower_leg_skin_20_fixed_joint: origin xyz=0.0234419 0.047990799999999986 -0.004952000000000012 rpy=-3.2055655013539e-06 -1.5001551303072311 -1.8675509241250052 -> xyz=0.023441900000000012 0.04799079999999998 -0.004952000000000012 rpy=-3.2055655013539e-06 -1.5001551303072311 -1.8675509241250052
- joint r_lower_leg_skin_21_fixed_joint: origin xyz=0.024270400000000004 0.04853779999999998 -0.024276999999999993 rpy=2.2967114952132173e-05 -1.555455138805717 -1.8741197231627162 -> xyz=0.02427040000000001 0.04853779999999998 -0.024276999999999993 rpy=2.2967114952132173e-05 -1.555455138805717 -1.8741197231627162
- joint r_lower_leg_skin_28_fixed_joint: origin xyz=0.04087215999999998 -0.0424399 -0.03275600000000001 rpy=3.1415808886539165 -1.5225246216918655 -0.9296810297631274 -> xyz=0.04087214999999999 -0.04244000000000002 -0.03275600000000001 rpy=3.1415808886539165 -1.5225246216918655 -0.9296810297631274
- joint r_lower_leg_skin_29_fixed_joint: origin xyz=0.03846637999999998 -0.04351590000000001 -0.05242000000000002 rpy=3.1415801704422774 -1.5342984156258153 -0.9154363466305139 -> xyz=0.038466369999999986 -0.04351600000000001 -0.05242000000000002 rpy=3.1415801704422774 -1.5342984156258153 -0.9154363466305139
- joint r_lower_leg_skin_31_fixed_joint: origin xyz=0.03914639999999998 -0.042270899999999986 0.006327000000000027 rpy=-6.583817471389409e-07 -1.4186494462021593 2.2085303298592955 -> xyz=0.03914637999999999 -0.04227099999999999 0.006327000000000027 rpy=-6.583817471389409e-07 -1.4186494462021593 2.2085303298592955
- joint r_lower_leg_skin_32_fixed_joint: origin xyz=0.045983029999999994 0.03258469999999997 -0.080733 rpy=-3.141590149878832 -1.5223828979770995 0.6459403808870791 -> xyz=0.045983010000000005 0.032584699999999966 -0.080733 rpy=-3.141590149878832 -1.5223828979770995 0.6459403808870791
- joint r_lower_leg_skin_35_fixed_joint: origin xyz=0.04774867999999998 -0.031231900000000007 -0.08011299999999999 rpy=-3.1415866827530343 -1.5175846733225289 -0.5415324864684377 -> xyz=0.047748659999999984 -0.031231999999999996 -0.08011299999999999 rpy=-3.1415866827530343 -1.5175846733225289 -0.5415324864684377
- joint r_lower_leg_skin_36_fixed_joint: origin xyz=0.05322409999999998 -0.015601800000000027 -0.088362 rpy=-3.141590341443774 -1.515872652806505 -0.2074073356601009 -> xyz=0.05322408999999999 -0.01560180000000004 -0.088362 rpy=-3.141590341443774 -1.515872652806505 -0.2074073356601009
- joint r_lower_leg_skin_37_fixed_joint: origin xyz=0.055257199999999985 0.0009643999999999764 -0.078318 rpy=-3.1415818045233417 -1.5231833689799856 0.007524505830633038 -> xyz=0.05525719999999999 0.0009643999999999903 -0.078318 rpy=-3.1415818045233417 -1.5231833689799856 0.007524505830633038
- joint r_lower_leg_skin_38_fixed_joint: origin xyz=0.04880468999999998 -0.03126290000000001 -0.060757000000000005 rpy=3.1415866519890927 -1.515729955403707 -0.5421535995897713 -> xyz=0.04880466999999999 -0.031263 -0.060757000000000005 rpy=3.1415866519890927 -1.515729955403707 -0.5421535995897713
- joint r_lower_leg_skin_3_fixed_joint: origin xyz=0.05157878999999999 0.030420499999999996 -0.0028429999999999844 rpy=0 -1.4295105408285231 -2.3039148418553874 -> xyz=0.051578780000000005 0.03042049999999999 -0.0028429999999999844 rpy=0 -1.4295105408285231 -2.3039148418553874
- joint r_lower_leg_skin_41_fixed_joint: origin xyz=0.05660089999999998 -0.015912900000000008 -0.049853999999999954 rpy=-3.1415919882511 -1.40681343597041 -0.24823308941290148 -> xyz=0.05660089999999999 -0.01591290000000002 -0.049853999999999954 rpy=-3.1415919882511 -1.40681343597041 -0.24823308941290148
- joint r_lower_leg_skin_42_fixed_joint: origin xyz=0.05701059999999998 0.000796199999999983 -0.059079999999999966 rpy=3.141589702392633 -1.4352475041611767 0.006879436515037955 -> xyz=0.057010599999999995 0.000796199999999983 -0.059079999999999966 rpy=3.141589702392633 -1.4352475041611767 0.006879436515037955
- joint r_lower_leg_skin_43_fixed_joint: origin xyz=0.04712543999999999 0.03236529999999998 -0.06136200000000003 rpy=-3.1415913662061943 -1.5384303823718677 0.6242175236666732 -> xyz=0.04712542 0.03236529999999998 -0.06136200000000003 rpy=-3.1415913662061943 -1.5384303823718677 0.6242175236666732
- joint r_lower_leg_skin_46_fixed_joint: origin xyz=0.05581569999999999 0.01721639999999998 -0.05018 rpy=-3.141589878093782 -1.4275988160283246 0.3256077108756132 -> xyz=0.0558156 0.01721639999999998 -0.05018 rpy=-3.141589878093782 -1.4275988160283246 0.3256077108756132
- joint r_lower_leg_skin_47_fixed_joint: origin xyz=0.052641649999999984 0.017638799999999975 -0.08886 rpy=3.141589635185034 -1.5169055940579301 0.26264042505774415 -> xyz=0.052641629999999995 0.01763889999999997 -0.08886 rpy=3.141589635185034 -1.5169055940579301 0.26264042505774415
- joint r_lower_leg_skin_49_fixed_joint: origin xyz=0.04113139 0.03243849999999996 -0.138859 rpy=-3.1415893475069225 -1.4899613569502461 0.7297635921130964 -> xyz=0.04113137 0.032438499999999953 -0.138859 rpy=-3.1415893475069225 -1.4899613569502461 0.7297635921130964
- joint r_lower_leg_skin_4_fixed_joint: origin xyz=0.05831029999999999 0.016783599999999996 0.007272000000000001 rpy=-2.986363594545861e-07 -1.2563674887550182 -2.7589238008709835 -> xyz=0.058310299999999995 0.016783599999999996 0.007272000000000001 rpy=-2.986363594545861e-07 -1.2563674887550182 -2.7589238008709835
- joint r_lower_leg_skin_50_fixed_joint: origin xyz=0.04301696299999999 0.03252729999999997 -0.11946899999999999 rpy=3.1415906959631426 -1.4990073263616448 0.6957840200808761 -> xyz=0.04301694700000001 0.03252729999999996 -0.11946899999999999 rpy=3.1415906959631426 -1.4990073263616448 0.6957840200808761
- joint r_lower_leg_skin_51_fixed_joint: origin xyz=0.05141583999999999 0.01775899999999997 -0.10820600000000002 rpy=-3.141588901786459 -1.5062847571686897 0.27207993571349487 -> xyz=0.051415829999999996 0.017758999999999962 -0.10820600000000002 rpy=-3.141588901786459 -1.5062847571686897 0.27207993571349487
- joint r_lower_leg_skin_52_fixed_joint: origin xyz=0.052998339999999984 0.001266399999999973 -0.11689500000000003 rpy=-3.141591640420276 -1.5031867442105085 0.010871726099408735 -> xyz=0.052998319999999995 0.0012663999999999592 -0.11689500000000003 rpy=-3.141591640420276 -1.5031867442105085 0.010871726099408735
- joint r_lower_leg_skin_53_fixed_joint: origin xyz=0.05207313999999998 -0.015433900000000028 -0.10765399999999997 rpy=3.1415906398667093 -1.5059530744712215 -0.21140732289166783 -> xyz=0.05207311999999999 -0.015433900000000042 -0.10765399999999997 rpy=3.1415906398667093 -1.5059530744712215 -0.21140732289166783
- joint r_lower_leg_skin_54_fixed_joint: origin xyz=0.045127099999999976 -0.03074890000000001 -0.11878700000000003 rpy=3.141588251928225 -1.4974514557145626 -0.5751153744726966 -> xyz=0.045127079999999986 -0.030749000000000026 -0.11878700000000003 rpy=3.141588251928225 -1.4974514557145626 -0.5751153744726966
- joint r_lower_leg_skin_55_fixed_joint: origin xyz=0.04350267899999998 -0.030488900000000027 -0.13814300000000007 rpy=3.1415890648626297 -1.4899578703820784 -0.5972199437885269 -> xyz=0.04350266299999999 -0.030489000000000016 -0.13814300000000007 rpy=3.1415890648626297 -1.4899578703820784 -0.5972199437885269
- joint r_lower_leg_skin_56_fixed_joint: origin xyz=0.049268409999999985 -0.015121000000000037 -0.1462179999999999 rpy=-3.141589204039199 -1.491248198275157 -0.22348447640041147 -> xyz=0.049268389999999995 -0.015121000000000051 -0.1462179999999999 rpy=-3.141589204039199 -1.491248198275157 -0.22348447640041147
- joint r_lower_leg_skin_5_fixed_joint: origin xyz=0.06365039999999998 0.00030939999999998746 -0.0019720000000000293 rpy=0 -1.3865221506831833 -3.1414716980716264 -> xyz=0.06365029999999999 0.00030940000000000134 -0.0019720000000000293 rpy=0 -1.3865221506831833 -3.1414716980716264
- joint r_lower_leg_skin_60_fixed_joint: origin xyz=0.04836967999999999 0.018055999999999968 -0.14693799999999996 rpy=-3.141591733372508 -1.4898596852742692 0.3029518719544257 -> xyz=0.04836967 0.01805599999999996 -0.14693799999999996 rpy=-3.141591733372508 -1.4898596852742692 0.3029518719544257
- joint r_lower_leg_skin_61_fixed_joint: origin xyz=0.051619539999999985 0.0014265999999999723 -0.13616899999999993 rpy=-3.141591009251115 -1.4960209708613401 0.013201427520491136 -> xyz=0.051619519999999995 0.0014265999999999723 -0.13616899999999993 rpy=-3.141591009251115 -1.4960209708613401 0.013201427520491136
- joint r_lower_leg_skin_6_fixed_joint: origin xyz=0.05208553999999999 0.03044339999999999 -0.022148999999999974 rpy=-3.1415892795257623 -1.4678512341064949 0.8374928890768587 -> xyz=0.05208552 0.03044339999999998 -0.022148999999999974 rpy=-3.1415892795257623 -1.4678512341064949 0.8374928890768587
- joint r_lower_leg_skin_9_fixed_joint: origin xyz=0.05982139999999998 0.01679719999999999 -0.03096199999999999 rpy=-3.1415920235620423 -1.3422475532506952 0.37929447771782354 -> xyz=0.0598214 0.016797299999999987 -0.03096199999999999 rpy=-3.1415920235620423 -1.3422475532506952 0.37929447771782354
- joint r_sole_fixed_joint: origin xyz=0.003500000000000003 0 0.0040000000000000036 rpy=-3.141592653589793 0 0 -> xyz=0.021450226059648816 0 0.006691276652475264 rpy=-3.1415926535897913 0.2617991810276664 0
- joint r_upper_leg_back_contact_fixed_joint: origin xyz=-0.051199800000000004 0 0.014599999999999946 rpy=0 1.5707963267948963 0 -> xyz=-0.05119989999999999 0 0.014599999999999946 rpy=0 1.5707963267948963 0
- joint torso_pitch: origin xyz=0 0.027046299999999992 0 rpy=1.5707963267948961 0 -1.5707963267948961 -> xyz=0 0.02693479999999999 0 rpy=1.5707963267948961 0 -1.5707963267948961
- joint torso_roll: origin xyz=0.027046299809264998 0.032 -0.05734460000000001 rpy=0 0 0 -> xyz=0.026934799809264998 0.032 -0.05734460000000001 rpy=0 0 0
